File: _autosave-ziol.kicad_pcb (KiCad board)
At the start: 2 copper layers, 82 parts, among them U1 Raspberry_Pi_Pico, U2 Raspberry_Pi_Pico

Commit message: Piece De Revolution
Parts:
- added J1: PJ324M, PJ324M:WENZHOU_PJ324M, F.Cu at (226.7, 47.5)
- added J2: PJ324M, PJ324M:WENZHOU_PJ324M, F.Cu at (213.0, 47.5)
- added J3: UJC-H-G-SMT-P6-TR, UJC-H-G-SMT-P6-TR:SAMESKY_UJC-H-G-SMT-P6-TR, F.Cu at (302.1, 24.7)
- added J4: Conn_01x06_Shielded, UJC-H-G-SMT-P6-TR:SAMESKY_UJC-H-G-SMT-P6-TR, F.Cu at (313.5, 43.7)
- added J5: UJC-H-G-SMT-P6-TR, UJC-H-G-SMT-P6-TR:SAMESKY_UJC-H-G-SMT-P6-TR, F.Cu at (218.5, 91.2)
- added J6: UJC-H-G-SMT-P6-TR, UJC-H-G-SMT-P6-TR:SAMESKY_UJC-H-G-SMT-P6-TR, F.Cu at (248.9, 51.3)
- added J7: Conn_01x06_Shielded, Connector_USB:USB_C_Receptacle_GCT_USB4125-xx-x-0190_6P_TopMnt_Horizontal, F.Cu at (345.8, 43.7)
Connections:
- D22 pad 1: Net-(D22-K) -> Net-(D21-K)
- D23 pad 1: Net-(D23-K) -> Net-(D21-K)
- D24 pad 1: Net-(D24-K) -> Net-(D21-K)
- D26 pad 1: Net-(D22-K) -> Net-(D21-K)
- D27 pad 1: Net-(D23-K) -> Net-(D21-K)
- D28 pad 1: Net-(D24-K) -> Net-(D21-K)
- D30 pad 1: Net-(D22-K) -> Net-(D21-K)
- D31 pad 1: Net-(D23-K) -> Net-(D21-K)
- D32 pad 1: Net-(D24-K) -> Net-(D21-K)
- D34 pad 1: Net-(D22-K) -> Net-(D21-K)
- D35 pad 1: Net-(D23-K) -> Net-(D21-K)
- D36 pad 1: Net-(D24-K) -> Net-(D21-K)
- D38 pad 1: Net-(D22-K) -> Net-(D21-K)
- D39 pad 1: Net-(D23-K) -> Net-(D21-K)
- D40 pad 1: Net-(D24-K) -> Net-(D21-K)
- U1 pad 21: unconnected-(U1-GPIO16-Pad21) -> Net-(U1-GPIO16)
- U1 pad 22: unconnected-(U1-GPIO17-Pad22) -> Net-(U1-GPIO17)
- U1 pad 23: unconnected-(U1-GND-Pad23) -> Net-(J5-CC2)
- U1 pad 24: unconnected-(U1-GPIO18-Pad24) -> Net-(J5-CC1)
- U1 pad 25: unconnected-(U1-GPIO19-Pad25) -> Net-(U1-GPIO19)
- U2 pad 1: unconnected-(U2-GPIO0-Pad1) -> Net-(U2-GPIO0)
- U2 pad 12: unconnected-(U2-GPIO9-Pad12) -> Net-(D21-K)
- U2 pad 13: unconnected-(U2-GND-Pad13) -> Net-(D21-K)
- U2 pad 14: unconnected-(U2-GPIO10-Pad14) -> Net-(D21-K)
- U2 pad 15: unconnected-(U2-GPIO11-Pad15) -> Net-(D21-K)
- U2 pad 17: Net-(D22-K) -> Net-(D21-K)
- U2 pad 18: unconnected-(U2-GND-Pad18) -> Net-(D21-K)
- U2 pad 19: Net-(D23-K) -> Net-(D21-K)
- U2 pad 2: unconnected-(U2-GPIO1-Pad2) -> Net-(U2-GPIO1)
- U2 pad 20: Net-(D24-K) -> Net-(D21-K)
- U2 pad 3: unconnected-(U2-GND-Pad3) -> Net-(J2-Pad1)
Routing:
- net (no net): track 0.00 -> 122.4 mm
