File: _autosave-ziol.kicad_sch (KiCad schematic)
At the start: 89 parts, among them J1 PJ324M, J2 PJ324M, J3 UJC-H-G-SMT-P6-TR, J4 Conn_01x06_Shielded, J5 UJC-H-G-SMT-P6-TR, J6 UJC-H-G-SMT-P6-TR, J7 Conn_01x06_Shielded, U1 Raspberry_Pi_Pico, U2 Raspberry_Pi_Pico

Commit message: Piece De Revolution
Parts:
- removed J1: PJ324M, PJ324M:WENZHOU_PJ324M, symbol PJ324M:PJ324M
- removed J3, J5, J6: UJC-H-G-SMT-P6-TR, UJC-H-G-SMT-P6-TR:SAMESKY_UJC-H-G-SMT-P6-TR, symbol UJC-H-G-SMT-P6-TR:UJC-H-G-SMT-P6-TR
- removed J4: Conn_01x06_Shielded, UJC-H-G-SMT-P6-TR:SAMESKY_UJC-H-G-SMT-P6-TR, symbol Connector_Generic_Shielded:Conn_01x06_Shielded
- removed J7: Conn_01x06_Shielded, Connector_USB:USB_C_Receptacle_GCT_USB4125-xx-x-0190_6P_TopMnt_Horizontal, symbol Connector_Generic_Shielded:Conn_01x06_Shielded
