File: ziol.kicad_pcb (KiCad board)
At the start: 2 copper layers, 82 parts, among them U1 Raspberry_Pi_Pico, U2 Raspberry_Pi_Pico

Commit message: Piece De Revolution
Parts:
- moved U1 201.7 mm to (129.8, 59.5)
- moved S12 5.70 mm to (85.5, 98.8)
- moved S15 5.70 mm to (85.5, 79.8)
- moved S16 5.70 mm to (104.5, 98.8)
- moved S18 5.70 mm to (104.5, 60.8)
- moved S19 5.70 mm to (104.5, 79.8)
- moved S20 5.70 mm to (123.5, 117.8)
- moved S8 5.70 mm to (66.5, 117.8)
- moved S13 5.70 mm to (85.5, 41.8)
- moved S14 5.70 mm to (85.5, 60.9)
- moved S17 5.70 mm to (104.5, 41.8)
Changed lines of the file:
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@@
 	(footprint "ScottoKeebs_MX:MX_PCB_1.00u"
 		(layer "F.Cu")
-		(at 66.525 123.525)
+		(at 66.525 117.825)
 		(descr "MX keyswitch PCB Mount Keycap 1.00u")
 		(tags "MX Keyboard Keyswitch Switch PCB Cutout Keycap 1.00u")
@@
 	(footprint "ScottoKeebs_MX:MX_PCB_1.00u"
 		(layer "F.Cu")
-		(at 85.525 66.55)
+		(at 85.525 60.85)
 		(descr "MX keyswitch PCB Mount Keycap 1.00u")
 		(tags "MX Keyboard Keyswitch Switch PCB Cutout Keycap 1.00u")
@@
 	(footprint "ScottoKeebs_MX:MX_PCB_1.00u"
 		(layer "F.Cu")
-		(at 104.525 66.525)
+		(at 104.525 60.825)
 		(descr "MX keyswitch PCB Mount Keycap 1.00u")
 		(tags "MX Keyboard Keyswitch Switch PCB Cutout Keycap 1.00u")
@@
 	(footprint "ScottoKeebs_MX:MX_PCB_1.00u"
 		(layer "F.Cu")
-		(at 104.525 47.525)
+		(at 104.525 41.825)
 		(descr "MX keyswitch PCB Mount Keycap 1.00u")
 		(tags "MX Keyboard Keyswitch Switch PCB Cutout Keycap 1.00u")
@@
 	(footprint "ScottoKeebs_MCU:Raspberry_Pi_Pico"
 		(layer "F.Cu")
-		(at 23.545 -111.91875)
+		(at 129.81 59.49)
 		(property "Reference" "U1"
 			(at 0 -32 0)
@@
 	(footprint "ScottoKeebs_MX:MX_PCB_1.00u"
 		(layer "F.Cu")
-		(at 104.525 85.525)
+		(at 104.525 79.825)
 		(descr "MX keyswitch PCB Mount Keycap 1.00u")
 		(tags "MX Keyboard Keyswitch Switch PCB Cutout Keycap 1.00u")
@@
 	(footprint "ScottoKeebs_MX:MX_PCB_1.00u"
 		(layer "F.Cu")
-		(at 85.525 104.525)
+		(at 85.525 98.825)
 		(descr "MX keyswitch PCB Mount Keycap 1.00u")
 		(tags "MX Keyboard Keyswitch Switch PCB Cutout Keycap 1.00u")
@@
 	(footprint "ScottoKeebs_MX:MX_PCB_1.00u"
 		(layer "F.Cu")
-		(at 104.525 104.525)
+		(at 104.525 98.825)
 		(descr "MX keyswitch PCB Mount Keycap 1.00u")
 		(tags "MX Keyboard Keyswitch Switch PCB Cutout Keycap 1.00u")
@@
 	(footprint "ScottoKeebs_MX:MX_PCB_1.00u"
 		(layer "F.Cu")
-		(at 85.525 85.525)
+		(at 85.525 79.825)
 		(descr "MX keyswitch PCB Mount Keycap 1.00u")
 		(tags "MX Keyboard Keyswitch Switch PCB Cutout Keycap 1.00u")
@@
 	(footprint "ScottoKeebs_MX:MX_PCB_1.00u"
 		(layer "F.Cu")
-		(at 85.525 47.525)
+		(at 85.525 41.825)
 		(descr "MX keyswitch PCB Mount Keycap 1.00u")
 		(tags "MX Keyboard Keyswitch Switch PCB Cutout Keycap 1.00u")
@@
 	(footprint "ScottoKeebs_MX:MX_PCB_1.00u"
 		(layer "F.Cu")
-		(at 123.525 123.525)
+		(at 123.525 117.825)
 		(descr "MX keyswitch PCB Mount Keycap 1.00u")
 		(tags "MX Keyboard Keyswitch Switch PCB Cutout Keycap 1.00u")
@@
 		)
 	)
+	(gr_poly
+		(pts
+			(xy 17.1 36.1) (xy 17.1 115.9) (xy 53.2 115.9) (xy 53.2 129.2) (xy 142.5 129.2) (xy 144.4 30.4) (xy 77.9 30.4)
+			(xy 77.9 13.3) (xy 57 13.3)
+		)
+		(stroke
+			(width 0.2)
+			(type solid)
+		)
+		(fill solid)
+		(layer "F.Cu")
+	)
 )
